File: agudo.kicad_pcb (KiCad board)
At the start: 2 copper layers, 28.8 x 54 mm, 49 parts, among them J1 Stomp_Connector, J2 Power_Connector, J3 Power_TOP, Q1 MMBF5457, Q2 MMBF5457, U1 TL072, U2 TL072

Commit message: updated to KiCad 6.0
Other:
- net class Default removed
- rule pad_to_mask_clearance: 0.05 -> 0
